Commit message: add material for visualization

File: robots/hand.gazebo.xacro (robot description, xacro)
@@ -1,7 +1,22 @@
 <?xml version='1.0' encoding='utf-8'?>
 <robot xmlns:xacro="http://www.ros.org/wiki/xacro" name="panda">
-	<gazebo reference="${ns}_hand"/>
-	<gazebo reference="${ns}_leftfinger"/>
-	<gazebo reference="${ns}_rightfinger"/>
+        <!-- LinkHand -->
+        <gazebo reference="${ns}_hand">
+            <material>Gazebo/Grey</material>
+            <mu1>0.2</mu1>
+            <mu2>0.2</mu2>
+        </gazebo>
+        <!-- LinkRightFinger -->
+        <gazebo reference="${ns}_rightfinger">
+            <material>Gazebo/Grey</material>
+            <mu1>0.2</mu1>
+            <mu2>0.2</mu2>
+        </gazebo>
+        <!-- LinkLeftFinger -->
+        <gazebo reference="${ns}_leftfinger">
+            <material>Gazebo/Grey</material>
+            <mu1>0.2</mu1>
+            <mu2>0.2</mu2>
+        </gazebo>
 	<transmission name="${ns}_finger_joint1_trans">
     <type>transmission_interface/SimpleTransmission</type>

File: robots/panda_arm.gazebo.xacro (robot description, xacro)
@@ -6,13 +6,58 @@
     </plugin>
   </gazebo>
-	<gazebo reference="${arm_id}_link0"/>
-	<gazebo reference="${arm_id}_link1"/>
-	<gazebo reference="${arm_id}_link2"/>
-	<gazebo reference="${arm_id}_link3"/>
-	<gazebo reference="${arm_id}_link4"/>
-	<gazebo reference="${arm_id}_link5"/>
-	<gazebo reference="${arm_id}_link6"/>
-	<gazebo reference="${arm_id}_link7"/>
-	<gazebo reference="${arm_id}_link8"/>
+ <!-- Link0 -->
+        <gazebo reference="${arm_id}_link0">
+            <material>Gazebo/Grey</material>
+            <mu1>0.2</mu1>
+            <mu2>0.2</mu2>
+        </gazebo>
+        <!-- Link1 -->
+        <gazebo reference="${arm_id}_link1">
+            <material>Gazebo/White</material>
+            <mu1>0.2</mu1>
+            <mu2>0.2</mu2>
+        </gazebo>
+        <!-- Link2 -->
+        <gazebo reference="${arm_id}_link2">
+            <material>Gazebo/White</material>
+            <mu1>0.2</mu1>
+            <mu2>0.2</mu2>
+        </gazebo>
+        <!-- Link3 -->
+        <gazebo reference="${arm_id}_link3">
+            <material>Gazebo/White</material>
+            <mu1>0.2</mu1>
+            <mu2>0.2</mu2>
+        </gazebo>
+        <!-- Link4 -->
+        <gazebo reference="${arm_id}_link4">
+            <material>Gazebo/White</material>
+            <mu1>0.2</mu1>
+            <mu2>0.2</mu2>
+        </gazebo>
+        <!-- Link5 -->
+        <gazebo reference="${arm_id}_link5">
+            <material>Gazebo/White</material>
+            <mu1>0.2</mu1>
+            <mu2>0.2</mu2>
+        </gazebo>
+        <!-- Link6 -->
+        <gazebo reference="${arm_id}_link6">
+            <material>Gazebo/White</material>
+            <mu1>0.2</mu1>
+            <mu2>0.2</mu2>
+        </gazebo>
+        <!-- Link7 -->
+        <gazebo reference="${arm_id}_link7">
+            <material>Gazebo/Grey</material>
+            <mu1>0.2</mu1>
+            <mu2>0.2</mu2>
+        </gazebo>
+        <!-- Link8 -->
+        <gazebo reference="${arm_id}_link8">
+            <material>Gazebo/Grey</material>
+            <mu1>0.2</mu1>
+            <mu2>0.2</mu2>
+        </gazebo>
 	 <transmission name="${arm_id}_joint1_trans">
     <type>transmission_interface/SimpleTransmission</type>
